Commit message: merge all the versions

File: catkin_ws/src/autominy_simulator/car_description/urdf/car.urdf (robot description, URDF)
Before this commit: robot car, 16 links, 15 joints
Links:
- added link camera_depth_frame
Joints:
- added joint camera_depth: type fixed, parent camera, child camera_depth_frame, origin rpy=-1.57079632679 0 -1.57079632679
- joint camera_joint: origin xyz=0.087 0 0.04 rpy=0 0.15 0 -> xyz=0.035 0 0.03 rpy=0 0 0

Commit message: manually apply marcels patch

File: catkin_ws/src/autominy_simulator/car_description/urdf/car.urdf (robot description, URDF)
Before this commit: robot car, 18 links, 17 joints
Links:
- added link chasi, mass 0.001; collision mesh filename=package://car_description/meshes/chasi.dae; visual mesh filename=package://car_description/meshes/chasi.dae
- link base_link: geometry 
Joints:
- removed joint base_link_board
- added joint base_chasi: type fixed, parent base_link, child chasi, origin xyz=0.135 0 0
- added joint chasi_board: type fixed, parent chasi, child board, origin xyz=-0.018 0 0.06
- joint frontwheel_steering_left: parent base_link -> chasi
- joint frontwheel_steering_right: parent base_link -> chasi
- joint rearwheel_left: parent base_link -> chasi
- joint rearwheel_right: parent base_link -> chasi
