Commit message: max friction

File: catkin_ws/src/autominy_simulator/car_description/urdf/car (copy).urdf (robot description, URDF)
Before this commit: robot car, 19 links, 18 joints
Links:
- link wheel_bl: geometry collision mesh filename=package://car_description/meshes/wheel.dae; visual mesh filename=package://car_description/meshes/wheel.dae
- link wheel_br: geometry collision mesh filename=package://car_description/meshes/wheel.dae; visual mesh filename=package://car_description/meshes/wheel.dae
- link wheel_fl: geometry collision mesh filename=package://car_description/meshes/wheel.dae; visual mesh filename=package://car_description/meshes/wheel.dae
- link wheel_fr: geometry collision mesh filename=package://car_description/meshes/wheel.dae; visual mesh filename=package://car_description/meshes/wheel.dae
